File: ElectronicsPCB/ElectronicsPCBv1.kicad_pcb (KiCad board)
At the start: 4 copper layers, 62.2 x 75.6 mm, 17 parts

Commit message: added mounting holes
Changed lines of the file:
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@@
 		)
 		(fp_text user "*"
-			(at 0 -1.4478 0)
+			(at 0 -1.4478 180)
+			(unlocked yes)
 			(layer "F.SilkS")
 			(effects
@@
 		)
 		(fp_text user "*"
-			(at 0.127 0 0)
+			(at 0.127 0 180)
+			(layer "F.Fab")
+			(effects
+				(font
+					(size 1 1)
+					(thickness 0.15)
+				)
+			)
+		)
+		(fp_text user "*"
+			(at 0.127 0 180)
 			(layer "F.Fab")
 			(effects
@@
 		(fp_text user "${REFERENCE}"
 			(at 3.81 8.89 90)
-			(unlocked yes)
-			(layer "F.Fab")
-			(effects
-				(font
-					(size 1 1)
-					(thickness 0.15)
-				)
-			)
-		)
-		(fp_text user "*"
-			(at 0.127 0 180)
 			(unlocked yes)
 			(layer "F.Fab")
@@
 			(layer "F.Fab")
 		)
+		(fp_text user "GND"
+			(at -12.065 -16.256 270)
+			(layer "F.SilkS")
+			(effects
+				(font
+					(size 0.64 0.64)
+					(thickness 0.15)
+				)
+			)
+		)
+		(fp_text user "GND"
+			(at -12.065 -16.256 270)
+			(layer "F.Fab")
+			(effects
+				(font
+					(size 0.64 0.64)
+					(thickness 0.15)
+				)
+			)
+		)
 		(pad "0" thru_hole circle
