File: ElectronicsPCB/ElectronicsPCB.kicad_pcb (KiCad board)
At the start: 2 copper layers, 62 x 92 mm, 37 parts

Commit message: final update to elec pcb hopefully
Parts:
- removed TEENSY: DEV-15583, ElectronicsFootprints:MODULE_DEV-15583
- added C10: 0.1µF, ElectronicsFootprints:CAP_CL10B_01uf_0603, F.Cu at (118.7, 57.3)
- added C11: 0.1µF, ElectronicsFootprints:CAP_CL10B_01uf_0603, F.Cu at (127.7, 57.1)
- added C12: 0.1µF, ElectronicsFootprints:CAP_CL10B_01uf_0603, F.Cu at (136.6, 57.1)
- added C6: 0.1µF, ElectronicsFootprints:CAP_CL10B_01uf_0603, F.Cu at (111.3, 73.2)
- added C8: 0.1µF, ElectronicsFootprints:CAP_CL10B_01uf_0603, F.Cu at (109.3, 82.6)
- added C9: 0.1µF, ElectronicsFootprints:CAP_CL10B_01uf_0603, F.Cu at (109.2, 54.8)
- added G***: LOGO, LOGO, F.Cu at (104.1, 60.8)
- added G***: LOGO, LOGO, F.Cu at (108.6, 59.8)
- added TEENSY 4.0: DEV-15583, ElectronicsFootprints:MODULE_DEV-15583, F.Cu at (142.7, 73.8)
- H1, H2, H3: footprint MountingHole:MountingHole_2.7mm -> MountingHole:MountingHole_3.2mm_M3
- moved TeensyC0.1 59.3 mm to (158.5, 84.6)
- moved 5V_LOW1 24.8 mm to (120.0, 41.0), turned to -90 degrees
- moved C3 2.53 mm to (145.2, 109.2)
- moved C4 2.53 mm to (143.2, 109.2)
- moved MAX3323EEPE 2.53 mm to (140.4, 111.1)
- moved C2 1.99 mm to (143.1, 102.2)
- moved C1 1.93 mm to (143.1, 98.5)
- moved G*** 1.35 mm to (143.1, 125.7)
- moved H2 1.28 mm to (120.2, 72.8)
- moved 5V_EXTRA 1.12 mm to (113.9, 57.6)
- moved H3 1.10 mm to (158.4, 89.5)
- moved CAMERA 0.76 mm to (123.0, 57.6)
- moved SAIL 0.76 mm to (140.9, 57.5)
- moved TAIL 0.61 mm to (132.0, 57.5)
- moved 5V_MID1 0.40 mm to (105.2, 54.9), turned to -90 degrees
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Connections:
- 5V_LOW1 pad 1: +5V_SYS -> GND
- 5V_LOW1 pad 2: GND -> +5V_SYS
- 5V_MID1 pad 1: +5V_SYS -> GND
- 5V_MID1 pad 2: GND -> +5V_SYS
- HEADERS1 pad 25: Extra41 -> unconnected-(HEADERS1-Pad25)
- HEADERS1 pad 6: TEENSY_3.3V -> unconnected-(HEADERS1-Pad6)
- TeensyC0.1 pad 1: +5V_SYS -> GND
- TeensyC0.1 pad 2: GND -> +5V_SYS
Routing:
- net Extra40: track 99.6 -> 47.1 mm
- net Extra41: track 60.9 -> 22.1 mm
- net TEENSY_3.3V: track 56.4 -> 22.3 mm
- net GND: track 22.1 -> 29.2 mm, vias 27 -> 18
- net XBeeRESET: track 51.4 -> 48.7 mm
- net TeensyTX: track 45.1 -> 42.8 mm
- net TeensyRX: track 46.8 -> 44.5 mm, vias 0 -> 1
- net VBAT: track 32.7 -> 35.0 mm
- net Net-(StepDownChip1-C2-): track 4.80 -> 2.86 mm
- net Net-(StepDownChip1-V-): track 4.94 -> 3.02 mm
- net +5V_SYS: track 85.8 -> 87.6 mm, vias 0 -> 1
- net Net-(StepDownChip1-C2+): track 4.40 -> 2.82 mm
- net VectorNavTX: track 22.6 -> 21.2 mm
- net Sail: track 39.4 -> 38.2 mm
- net Extra3: track 50.3 -> 49.2 mm
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Other:
- board text added: "3.3V_BULK"
- board text added: "3.3V_MID"
- board text added: "5V_BULK1"
- board text added: "5V_BULK2"
- board text added: "5V_MID"
- board text added: "C7"
- board text added: "Controls PCB FA25/SP26 Liya Mei Jonah Conolly"
- board text added: "X"
- board text removed: "Controls PCB Fall 2025 Liya Mei Jonah Conolly"
