File: ElectronicsPCB/ElectronicsPCB.kicad_pcb (KiCad board)
At the start: 2 copper layers, 62 x 92 mm, 45 parts

Commit message: half done silkscreen
Parts:
- moved G*** 1.22 mm to (120.5, 76.9)
- moved G*** 0.79 mm to (118.5, 81.4)
Routing:
- net Tail: track 44.6 -> 43.8 mm
- net Camera: track 51.0 -> 50.2 mm
- net 2: track 26.0 -> 25.2 mm
- net Sail: track 38.2 -> 37.5 mm
- net 12: track 26.7 -> 27.5 mm
- net Extra40: track 47.1 -> 46.4 mm
- net XBeeRESET: track 48.7 -> 48.2 mm
Other:
- board text added: "+3.3V_SYS"
- board text added: "+3.3V_T"
- board text added: "ON_OFF"
- board text added: "PGM"

Commit message: series of changes
Parts:
- added 3.3V_BULK1: 220uf, ElectronicsFootprints:CAP_87510_220uf, F.Cu at (75.7, 118.5)
- added 5V_BULK3: 1000uf, ElectronicsFootprints:CAP_EEE1A_1000uf, F.Cu at (52.6, 107.2)
- added 5V_BULK4: 1000uf, ElectronicsFootprints:CAP_EEE1A_1000uf, F.Cu at (52.6, 119.1)
- added 5V_LOW2: 0.1uf, ElectronicsFootprints:CAP_CL10B_01uf_0603, F.Cu at (75.4, 77.6)
- added 5V_MID2: 22uf, ElectronicsFootprints:CAP_CL32A_22uf_1210, F.Cu at (76.3, 74.2)
- added 5V_SYS2: Conn_02x03_Counter_Clockwise, Connector_Molex:Molex_Mini-Fit_Jr_5566-06A_2x03_P4.20mm_Vertical, F.Cu at (61.3, 88.4)
- added EXTRA1: B4B-XH-A, ElectronicsFootprints:B4B-XH-A, F.Cu at (33.0, 120.9)
- added JIB1: B3B-XH-A, ElectronicsFootprints:B3B-XH-A, F.Cu at (46.0, 60.5)
- added JIB2: B3B-XH-A, ElectronicsFootprints:B3B-XH-A, F.Cu at (34.5, 77.0)
- renumbered 5V_SYS to 5V_SYS1
Connections:
- 5V_BULK1 pad 1: +5V_SYS -> +5V_SYS1
- 5V_BULK2 pad 1: +5V_SYS -> +5V_SYS1
- 5V_LOW1 pad 2: +5V_SYS -> +5V_SYS1
- 5V_MID1 pad 2: +5V_SYS -> +5V_SYS1
- C10 pad 1: +5V_SYS -> +5V_SYS1
- C11 pad 1: +5V_SYS -> +5V_SYS2
- C12 pad 1: +5V_SYS -> +5V_SYS1
- C9 pad 1: +5V_SYS -> +5V_SYS2
- HEADERS1 pad 2: +5V_SYS -> +5V_SYS1
- HEADERS1 pad 21: Extra3 -> JIB1
- HEADERS1 pad 23: Extra40 -> JIB2
- TeensyC0.1 pad 2: +5V_SYS -> +5V_SYS1
Routing:
- added copper zone on F.Cu, net +5V_SYS1
- removed copper zone on F.Cu, net +5V_SYS
