File: PowerDistributionPCB/untitled.kicad_sch (KiCad schematic)
At the start: 0 parts

Commit message: added relays and usb port
Changed lines of the file:
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@@
 	)
 	(hierarchical_label "Out"
-		(shape input)
+		(shape output)
 		(at 184.15 50.8 0)
 		(effects
@@
 		(dnp no)
 		(fields_autoplaced yes)
-		(property "Reference" "#PWR01"
+		(property "Reference" "#PWR"
 			(at 177.8 76.2 0)
 			(effects
@@
 		)
 		(instances
-			(project ""
-				(path "/b27c75df-6223-4cc6-be69-062c2b02d5c6/64db8257-fd15-498a-b60d-52dd4c6b0385"
+			(project "PowerDistributionPCB"
+				(path "/b27c75df-6223-4cc6-be69-062c2b02d5c6/4aa10ec7-4b36-4cde-a760-c4500e70a751"
 					(reference "#PWR01")
 					(unit 1)
 				)
-				(path "/b27c75df-6223-4cc6-be69-062c2b02d5c6/bfd015dc-a1f5-42ba-b972-f7703fed8888"
-					(reference "#PWR?")
-					(unit 1)
-				)
