File: PowerDistributionPCB/3VSTEPDOWN.kicad_sch (KiCad schematic)
At the start: 0 parts

Commit message: more things added to power
Parts:
- added C? (x4): C, symbol Device:C
- added L?: L, symbol Device:L
- added R? (x2): R, symbol Device:R
- added U?: AP63203WU, Package_TO_SOT_SMD:TSOT-23-6, symbol Regulator_Switching:AP63203WU
Connections:
- new net: R?.1, R?.1, U?.2 (EN)
- new net: C?.2, L?.1, U?.5 (SW)
- new net: C?.1, U?.6 (BST)
- new net +3.3V: C?.1, C?.1, L?.2, U?.1 (FB)
- new net +BATT: C?.1, R?.2, U?.3 (IN)
- new net GND: C?.2, C?.2, C?.2, R?.2, U?.4 (GND)

Commit message: finished reverse polarity and updated 3.3V stepdown
Parts:
- C1: renamed from C?; value C -> 10µF
- C2: renamed from C?; value C -> 0.1µF
- C3, C4: renamed from C?; value C -> 22µF
- L1: renamed from L?; value L -> 4.7µH
- R1, R2: renamed from R?; value R -> 100k
Changed lines of the file:
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@@
 		(dnp no)
 		(fields_autoplaced yes)
-		(property "Reference" "R?"
+		(property "Reference" "R2"
 			(at 119.38 82.5499 0)
 			(effects
@@
 			)
 		)
-		(property "Value" "R"
+		(property "Value" "100k"
 			(at 119.38 85.0899 0)
 			(effects
@@
 			(project ""
 				(path "/b27c75df-6223-4cc6-be69-062c2b02d5c6/079a49e6-596e-4e19-9f4e-bda307b8342c"
-					(reference "R?")
+					(reference "R2")
 					(unit 1)
 				)
@@
 		(dnp no)
 		(fields_autoplaced yes)
-		(property "Reference" "C?"
+		(property "Reference" "C4"
 			(at 193.04 85.0899 0)
 			(effects
@@
 			)
 		)
-		(property "Value" "C"
+		(property "Value" "22µF"
 			(at 193.04 87.6299 0)
 			(effects
@@
 			(project ""
 				(path "/b27c75df-6223-4cc6-be69-062c2b02d5c6/079a49e6-596e-4e19-9f4e-bda307b8342c"
-					(reference "C?")
+					(reference "C4")
 					(unit 1)
 				)
@@
 		(dnp no)
 		(fields_autoplaced yes)
-		(property "Reference" "R?"
+		(property "Reference" "R1"
 			(at 119.38 71.1199 0)
 			(effects
@@
 			)
 		)
-		(property "Value" "R"
+		(property "Value" "100k"
 			(at 119.38 73.6599 0)
 			(effects
@@
 			(project ""
 				(path "/b27c75df-6223-4cc6-be69-062c2b02d5c6/079a49e6-596e-4e19-9f4e-bda307b8342c"
-					(reference "R?")
+					(reference "R1")
 					(unit 1)
 				)
@@
 		(dnp no)
 		(fields_autoplaced yes)
-		(property "Reference" "C?"
+		(property "Reference" "C1"
 			(at 107.95 80.0099 0)
 			(effects
@@
 			)
 		)
-		(property "Value" "C"
+		(property "Value" "10µF"
 			(at 107.95 82.5499 0)
 			(effects
@@
 			(project ""
 				(path "/b27c75df-6223-4cc6-be69-062c2b02d5c6/079a49e6-596e-4e19-9f4e-bda307b8342c"
-					(reference "C?")
+					(reference "C1")
 					(unit 1)
 				)
@@
 		(dnp no)
 		(fields_autoplaced yes)
-		(property "Reference" "C?"
+		(property "Reference" "C2"
 			(at 163.83 72.39 90)
 			(effects
@@
 			)
 		)
-		(property "Value" "C"
+		(property "Value" "0.1µF"
 			(at 163.83 74.93 90)
 			(effects
@@
 			(project ""
 				(path "/b27c75df-6223-4cc6-be69-062c2b02d5c6/079a49e6-596e-4e19-9f4e-bda307b8342c"
-					(reference "C?")
+					(reference "C2")
 					(unit 1)
 				)
@@
 		(dnp no)
 		(fields_autoplaced yes)
-		(property "Reference" "C?"
+		(property "Reference" "C3"
 			(at 182.88 85.0899 0)
 			(effects
@@
 			)
 		)
-		(property "Value" "C"
+		(property "Value" "22µF"
 			(at 182.88 87.6299 0)
 			(effects
@@
 			(project ""
 				(path "/b27c75df-6223-4cc6-be69-062c2b02d5c6/079a49e6-596e-4e19-9f4e-bda307b8342c"
-					(reference "C?")
+					(reference "C3")
 					(unit 1)
 				)
@@
 		(dnp no)
 		(fields_autoplaced yes)
-		(property "Reference" "L?"
+		(property "Reference" "L1"
 			(at 172.72 72.39 90)
 			(effects
@@
 			)
 		)
-		(property "Value" "L"
+		(property "Value" "4.7µH"
 			(at 172.72 74.93 90)
 			(effects
@@
 			(project ""
 				(path "/b27c75df-6223-4cc6-be69-062c2b02d5c6/079a49e6-596e-4e19-9f4e-bda307b8342c"
-					(reference "L?")
-					(unit 1)
-				)
+					(reference "L1")
+					(unit 1)
+				)
