File: PowerDistributionPCB/Reverse_Polarity.kicad_sch (KiCad schematic)
At the start: 0 parts

Commit message: finished reverse polarity and updated 3.3V stepdown
Parts:
- added D1: MMSZ5242BS-7-F, symbol Device:D_Zener
- added Q?: AOD4185, TO252_AOS, symbol CU_Sail:AOD4185
- added R1, R2: 10k, symbol Device:R
Connections:
- new net: D1.2 (A), Q?.1 (G), R1.2, R2.2
- new net Batt_Vin: D1.1 (K), Q?.3 (S), R1.1
- new net GND: R2.1
- new net Sys_Vin: Q?.2 (D)
