File: PowerDistributionPCB/Relay.kicad_sch (KiCad schematic)
At the start: 7 parts, among them K2 RT314F05(gen), Q2 MMBT2222A, Q6 MMBT2222A

Commit message: fixing relay stuff
Connections:
- net VIN: now also K2.12.1, K2.12.2; no longer K2.11.1, K2.11.2
- new net: K2.11.1, K2.11.2
Changed lines of the file:
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@@
-	)
-	(junction
-		(at 161.29 77.47)
-		(diameter 0)
-		(color 0 0 0 0)
 	)
 	(junction
@@
 	)
 	(no_connect
-		(at 184.15 76.2)
+		(at 161.29 78.74)
 	)
 	(wire
@@
 		(pts
 			(xy 184.15 82.55) (xy 184.15 80.01)
-		)
-		(stroke
-			(width 0)
-			(type default)
-		)
-	)
-	(wire
-		(pts
-			(xy 160.02 77.47) (xy 161.29 77.47)
 		)
 		(stroke
@@
 	(hierarchical_label "VIN"
 		(shape input)
-		(at 160.02 77.47 180)
+		(at 184.15 74.93 0)
 		(effects
 			(font
 				(size 1.27 1.27)
 			)
-			(justify right)
-		)
-	)
+			(justify left)
+		)
+	)
