File: PowerDistributionPCB/PowerDistributionPCB.kicad_pcb (KiCad board)
At the start: 4 copper layers, 96 x 125.6 mm, 93 parts, among them K1 RT314F05(gen), K2 RT314F05(gen), K3 RT314F05(gen), K4 RT314F05(gen), Q1 AOD4185, Q10 MMBT2222A, Q11 MMBT2222A, Q12 MMBT2222A, Q2 MMBT2222A, Q6 MMBT2222A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

Commit message: final power pcb changes
Parts:
- C2b1, Cboot1: footprint Capacitor_SMD:C_0201_0603Metric_Pad0.64x0.40mm_HandSolder -> Capacitor_SMD:C_0402_1005Metric
- Cff1: footprint Capacitor_SMD:C_0201_0603Metric_Pad0.64x0.40mm_HandSolder -> Capacitor_SMD:C_0402_1005Metric_Pad0.74x0.62mm_HandSolder
- Main_Bulk: footprint Capacitor_SMD:C_1210_3225Metric_Pad1.33x2.70mm_HandSolder -> CUSail:WCAP-PSLP_6.3X7.7_DXL_
- moved Main_Bulk 1.80 mm to (125.0, 38.4), turned to 180 degrees
- moved G*** 1.79 mm to (134.4, 45.0)
- moved Cff1 0.10 mm to (93.9, 52.4)
Routing:
- net Sys_Vin: track 3.86 -> 4.09 mm, vias 13 -> 15
