File: Switchbox/Switchbox.kicad_sch (KiCad schematic)
At the start: 33 parts, among them J1 USB-C_connector, SW1 SW_SPDT, SW2 SW_SPDT, SW3 SW_SPDT, SW4 SW_SPDT, SW5 SW_SPST_LED, SW6 SW_SPDT_BOX, U2 AP63203WU

Commit message: arranged items in PCB editor- but I ran out of footprint downloads
Parts:
- C1: footprint (none) -> switchbox_footprints:CAPC1005X70N
- C2: footprint (none) -> switchbox_footprints:CAPC0603X33N
- C3, C4: footprint (none) -> switchbox_footprints:CAPC3216X190N
- C5: footprint ElectronicsFootprints:CAP_CL10B_01uf_0603 -> switchbox_footprints:CAPC0603X33N
Changed lines of the file:
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@@
 			)
 		)
-		(property "Footprint" "ElectronicsFootprints:CAP_CL10B_01uf_0603"
+		(property "Footprint" "switchbox_footprints:CAPC0603X33N"
 			(at 171.1452 127 0)
 			(effects
@@
 			)
 		)
-		(property "Footprint" ""
+		(property "Footprint" "switchbox_footprints:CAPC3216X190N"
 			(at 188.9252 57.15 0)
 			(effects
@@
 			)
 		)
-		(property "Footprint" ""
+		(property "Footprint" "switchbox_footprints:CAPC0603X33N"
 			(at 165.1 46.0248 0)
 			(effects
@@
 			)
 		)
-		(property "Footprint" ""
+		(property "Footprint" "switchbox_footprints:CAPC1005X70N"
 			(at 121.6152 52.07 0)
 			(effects
@@
 			)
 		)
-		(property "Footprint" ""
+		(property "Footprint" "switchbox_footprints:CAPC3216X190N"
 			(at 178.7652 57.15 0)
 			(effects

Commit message: changed footprints for big red button + switches into 4/3 pin headers
Parts:
- SW1, SW2, SW3, SW4, SW6: footprint switchbox_footprints:SW_SPDT -> switchbox_footprints:3_pin_header
- SW5: footprint switchbox_footprints:SPST_BUTTON_1190 -> switchbox_footprints:4_pin_header
Changed lines of the file:
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@@
 			)
 		)
-		(property "Footprint" "switchbox_footprints:SW_SPDT"
+		(property "Footprint" "switchbox_footprints:3_pin_header"
 			(at 72.39 50.8 0)
 			(effects
@@
 			)
 		)
-		(property "Footprint" "switchbox_footprints:SW_SPDT"
+		(property "Footprint" "switchbox_footprints:3_pin_header"
 			(at 40.64 88.9 0)
 			(effects
@@
 			)
 		)
-		(property "Footprint" "switchbox_footprints:SW_SPDT"
+		(property "Footprint" "switchbox_footprints:3_pin_header"
 			(at 40.64 119.38 0)
 			(effects
@@
 			)
 		)
-		(property "Footprint" "switchbox_footprints:SPST_BUTTON_1190"
+		(property "Footprint" "switchbox_footprints:4_pin_header"
 			(at 90.17 180.34 0)
 			(effects
@@
 			)
 		)
-		(property "Footprint" "switchbox_footprints:SW_SPDT"
+		(property "Footprint" "switchbox_footprints:3_pin_header"
 			(at 40.64 104.14 0)
 			(effects
@@
 			)
 		)
-		(property "Footprint" "switchbox_footprints:SW_SPDT"
+		(property "Footprint" "switchbox_footprints:3_pin_header"
 			(at 40.64 71.12 0)
 			(effects

Commit message: finished all the footprints
Parts:
- C6: footprint ElectronicsFootprints:CAP_C3225_47uf_1210 -> switchbox_footprints:CAPC2012X145N
- C7: value 100nF -> 0.1 uF; footprint (none) -> switchbox_footprints:CAPC0603X33N
Changed lines of the file:
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@@
 			)
 		)
-		(property "Value" "100nF"
+		(property "Value" "0.1 uF"
 			(at 79.756 169.672 0)
 			(effects
@@
 			)
 		)
-		(property "Footprint" ""
+		(property "Footprint" "switchbox_footprints:CAPC0603X33N"
 			(at 77.1652 172.72 0)
 			(effects
@@
 			)
 		)
-		(property "Footprint" "ElectronicsFootprints:CAP_C3225_47uf_1210"
+		(property "Footprint" "switchbox_footprints:CAPC2012X145N"
 			(at 177.4952 127 0)
 			(effects

Commit message: moving around components
Parts:
- D1, D2, D3, D4, D5, D6: footprint LED_THT:LED_D5.0mm -> switchbox_footprints:2_pin_header
Changed lines of the file:
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@@
 			)
 		)
-		(property "Footprint" "LED_THT:LED_D5.0mm"
+		(property "Footprint" "switchbox_footprints:2_pin_header"
 			(at 59.69 144.78 0)
 			(effects
@@
 			)
 		)
-		(property "Footprint" "LED_THT:LED_D5.0mm"
+		(property "Footprint" "switchbox_footprints:2_pin_header"
 			(at 59.69 121.92 0)
 			(effects
@@
 			)
 		)
-		(property "Footprint" "LED_THT:LED_D5.0mm"
+		(property "Footprint" "switchbox_footprints:2_pin_header"
 			(at 59.69 106.68 0)
 			(effects
@@
 			)
 		)
-		(property "Footprint" "LED_THT:LED_D5.0mm"
+		(property "Footprint" "switchbox_footprints:2_pin_header"
 			(at 59.69 91.44 0)
 			(effects
@@
 			)
 		)
-		(property "Footprint" "LED_THT:LED_D5.0mm"
+		(property "Footprint" "switchbox_footprints:2_pin_header"
 			(at 59.69 73.66 0)
 			(effects
@@
 			)
 		)
-		(property "Footprint" "LED_THT:LED_D5.0mm"
+		(property "Footprint" "switchbox_footprints:2_pin_header"
 			(at 59.69 133.35 0)
 			(effects
