File: Switchbox/Switchbox.kicad_pcb (KiCad board)
At the start: 2 copper layers, 90 x 68 mm, 37 parts, among them J1 USB-C_connector, SW1 SW_SPDT, SW2 SW_SPDT, SW3 SW_SPDT, SW4 SW_SPDT, SW5 SW_SPST_LED, SW6 SW_SPDT_BOX, U2 AP63203WU

Commit message: Resolved edge cut error
Parts:
- moved C5 0.10 mm to (120.8, 125.1)
Routing:
- net Net-(SW5-A): track 23.2 -> 19.4 mm
- net GND: track 215.0 -> 212.9 mm
Other:
- outline, holes or cut-outs redrawn
- board text removed: "${REFERENCE}"
Changed lines of the file:
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@@
 			(at 0.53 -0.77 90)
 			(layer "F.SilkS")
+			(hide yes)
 			(effects
 				(font
@@
 			(at -0.46 -1.32 0)
 			(layer "F.SilkS")
+			(hide yes)
 			(effects
 				(font
@@
 			(at -1.11 -1.55 0)
 			(layer "F.SilkS")
+			(hide yes)
 			(effects
 				(font
@@
 			(at 0.53 -0.77 90)
 			(layer "F.SilkS")
+			(hide yes)
 			(effects
 				(font
@@
 			(at 3.81 2.37 0)
 			(layer "F.Fab")
+			(hide yes)
 			(effects
 				(font
@@
 	(footprint "switchbox_footprints:CAPC0603X33N"
 		(layer "F.Cu")
-		(at 120.719 125)
+		(at 120.76 125.09)
 		(property "Reference" "C5"
 			(at 0.53 -0.77 0)
 			(layer "F.SilkS")
+			(hide yes)
 			(effects
 				(font
@@
 			(at 0.24 -0.95 0)
 			(layer "F.SilkS")
+			(hide yes)
 			(effects
 				(font
@@
 			(at -1.11 -1.55 0)
 			(layer "F.SilkS")
+			(hide yes)
 			(effects
 				(font
@@
 	)
 	(gr_line
-		(start 111 85)
-		(end 193 85)
-		(stroke
-			(width 0.0381)
-			(type default)
-		)
-		(layer "Edge.Cuts")
-	)
-	(gr_line
 		(start 103 153)
 		(end 193 153)
@@
 		(layer "Edge.Cuts")
 	)
-	(gr_text "${REFERENCE}"
-		(at 168.65 105.15 0)
-		(layer "F.Fab")
-		(effects
-			(font
-				(size 1 1)
-				(thickness 0.15)
-			)
-		)
-	)
-	(gr_text "${REFERENCE}"
-		(at 168.65 105.15 0)
-		(layer "F.Fab")
-		(effects
-			(font
-				(size 1 1)
-				(thickness 0.15)
-			)
-		)
-	)
 	(segment
 		(start 181 107)
@@
 	)
 	(segment
-		(start 132.9 123)
-		(end 133 123.1)
+		(start 120.775 128.248)
+		(end 121.041 127.982)
 		(width 0.127)
 		(layer "F.Cu")
@@
 	)
 	(segment
-		(start 121.9 124.1)
-		(end 121 125)
+		(start 165.054 143)
+		(end 165.054 147.5)
 		(width 0.127)
 		(layer "F.Cu")
@@
 	)
 	(segment
-		(start 121 125.2)
-		(end 120.775 125.425)
+		(start 120.775 128.248)
+		(end 118.647 128.248)
 		(width 0.127)
 		(layer "F.Cu")
@@
 	)
 	(segment
-		(start 121.9 123)
-		(end 132.9 123)
+		(start 163.4 143)
+		(end 162.8 142.4)
 		(width 0.127)
 		(layer "F.Cu")
@@
 	)
 	(segment
-		(start 120.775 128.248)
-		(end 118.647 128.248)
+		(start 121.9 123)
+		(end 121.9 124.231)
 		(width 0.127)
 		(layer "F.Cu")
@@
 	(segment
 		(start 165.054 143)
-		(end 165.054 147.5)
+		(end 163.4 143)
 		(width 0.127)
 		(layer "F.Cu")
@@
 	)
 	(segment
-		(start 118.647 128.248)
-		(end 114.585 132.31)
+		(start 123.15 123.07)
+		(end 123.08 123)
 		(width 0.127)
 		(layer "F.Cu")
@@
 	)
 	(segment
-		(start 121.9 123)
-		(end 121.9 124.1)
+		(start 121.041 127.982)
+		(end 121.041 125.09)
 		(width 0.127)
 		(layer "F.Cu")
@@
 	)
 	(segment
-		(start 163.4 143)
-		(end 162.8 142.4)
+		(start 118.647 128.248)
+		(end 114.585 132.31)
 		(width 0.127)
 		(layer "F.Cu")
@@
 	)
 	(segment
-		(start 120.775 125.425)
-		(end 120.775 128.248)
+		(start 123.75 123.07)
+		(end 123.15 123.07)
 		(width 0.127)
 		(layer "F.Cu")
@@
 	)
 	(segment
-		(start 165.054 143)
-		(end 163.4 143)
+		(start 123.08 123)
+		(end 121.9 123)
 		(width 0.127)
 		(layer "F.Cu")
@@
 	)
 	(segment
-		(start 121 125)
-		(end 121 125.2)
+		(start 121.9 124.231)
+		(end 121.041 125.09)
 		(width 0.127)
 		(layer "F.Cu")
@@
 	)
 	(via
-		(at 162.8 142.4)
+		(at 123.75 123.07)
 		(size 0.6)
 		(drill 0.3)
@@
 	)
 	(via
-		(at 177 148.4)
+		(at 162.8 142.4)
 		(size 0.6)
 		(drill 0.3)
@@
 	)
 	(via
-		(at 133 123.1)
+		(at 177 148.4)
 		(size 0.6)
 		(drill 0.3)
@@
 	)
 	(segment
+		(start 133 119.65)
+		(end 141.5 128.15)
+		(width 0.127)
+		(layer "B.Cu")
+		(net 6)
+	)
+	(segment
 		(start 177 131)
 		(end 173 135)
@@
 	)
 	(segment
+		(start 133 119.65)
+		(end 129.58 123.07)
+		(width 0.127)
+		(layer "B.Cu")
+		(net 6)
+	)
+	(segment
+		(start 157.22 111.5)
+		(end 152.14 106.42)
+		(width 0.127)
+		(layer "B.Cu")
+		(net 6)
+	)
+	(segment
 		(start 163.0085 89.2085)
 		(end 164.1 90.3)
@@
 	(segment
 		(start 141.5 128.15)
-		(end 133 119.65)
+		(end 141.5 131)
 		(width 0.127)
 		(layer "B.Cu")
@@
 	)
 	(segment
-		(start 141.5 131)
-		(end 141.5 128.15)
-		(width 0.127)
-		(layer "B.Cu")
-		(net 6)
-	)
-	(segment
 		(start 153.2 131.125)
 		(end 153.2 134.61)
@@
 	)
 	(segment
-		(start 162.8 142.4)
-		(end 165 140.2)
+		(start 129.58 123.07)
+		(end 123.75 123.07)
 		(width 0.127)
 		(layer "B.Cu")
@@
 	)
 	(segment
-		(start 133 123.1)
-		(end 133 119.65)
-		(width 0.127)
-		(layer "B.Cu")
-		(net 6)
-	)
-	(segment
-		(start 152.14 106.42)
-		(end 157.22 111.5)
+		(start 162.8 142.4)
+		(end 165 140.2)
 		(width 0.127)
 		(layer "B.Cu")
@@
 	)
 	(segment
-		(start 150.5 99.5)
-		(end 149.5 100.5)
-		(width 0.127)
-		(layer "F.Cu")
-		(net 7)
-	)
-	(segment
 		(start 118.35 123)
-		(end 120.1 123)
+		(end 115 119.65)
 		(width 0.127)
 		(layer "F.Cu")
@@
 	)
 	(segment
-		(start 115 119.65)
-		(end 118.35 123)
+		(start 150.5 99.5)
+		(end 149.5 100.5)
 		(width 0.127)
 		(layer "F.Cu")
@@
 	)
 	(segment
-		(start 120.1 124.662)
-		(end 120.438 125)
+		(start 120.479 123.379)
+		(end 120.1 123)
 		(width 0.127)
 		(layer "F.Cu")
@@
 	)
 	(segment
-		(start 149.5 106.2)
-		(end 128.45 106.2)
+		(start 120.479 125.09)
+		(end 120.479 123.379)
 		(width 0.127)
 		(layer "F.Cu")
@@
 	)
 	(segment
-		(start 120.438 123.338)
-		(end 120.1 123)
+		(start 149.5 106.2)
+		(end 128.45 106.2)
 		(width 0.127)
 		(layer "F.Cu")
@@
 	(segment
 		(start 120.1 123)
-		(end 120.1 124.662)
+		(end 118.35 123)
 		(width 0.127)
 		(layer "F.Cu")
@@
 	)
 	(segment
-		(start 151.5 103)
-		(end 151.536836 102.963164)
-		(width 0.127)
-		(layer "B.Cu")
-		(net 7)
-	)
-	(segment
 		(start 149.5 100.5)
 		(end 149.5 106.2)
@@
 	)
 	(segment
-		(start 120.19 133.19)
-		(end 120.775 132.605)
-		(width 0.127)
-		(layer "F.Cu")
-		(net 48)
-	)
-	(segment
-		(start 120.19 133.5)
-		(end 120.19 133.19)
-		(width 0.127)
-		(layer "F.Cu")
-		(net 48)
-	)
-	(segment
-		(start 108.0305 131.3645)
-		(end 111.1395 131.3645)
+		(start 113.275 133.5)
+		(end 120.19 133.5)
 		(width 0.127)
 		(layer "F.Cu")
@@
 	)
 	(segment
-		(start 120.775 132.605)
+		(start 120.19 129.395)
 		(end 120.775 128.81)
 		(width 0.127)
@@
 	)
 	(segment
-		(start 114 136)
-		(end 119 136)
+		(start 108.085 133.31)
+		(end 111.085 133.31)
 		(width 0.127)
 		(layer "F.Cu")
@@
 	)
 	(segment
-		(start 112.085 132.31)
-		(end 112.085 134.085)
-		(width 0.127)
-		(layer "F.Cu")
-		(net 48)
-	)
-	(segment
-		(start 119 136)
-		(end 120.19 134.81)
+		(start 120.19 133.5)
+		(end 120.19 129.395)
 		(width 0.127)
 		(layer "F.Cu")
@@
 	)
 	(segment
-		(start 107.085 132.31)
-		(end 108.0305 131.3645)
+		(start 112.085 132.31)
+		(end 113.275 133.5)
 		(width 0.127)
 		(layer "F.Cu")
@@
 	)
 	(segment
-		(start 111.1395 131.3645)
+		(start 111.085 133.31)
 		(end 112.085 132.31)
 		(width 0.127)
@@
 	)
 	(segment
-		(start 112.085 134.085)
-		(end 114 136)
-		(width 0.127)
-		(layer "F.Cu")
-		(net 48)
-	)
-	(segment
-		(start 120.19 134.81)
-		(end 120.19 133.5)
+		(start 107.085 132.31)
+		(end 108.085 133.31)
 		(width 0.127)
 		(layer "F.Cu")
@@
 		(polygon
 			(pts
-				(xy 95 155) (xy 95 83) (xy 200.5 82.5) (xy 201.5 155)
+				(xy 98.65 81.15) (xy 98.75 158.17) (xy 196.05 158.75) (xy 197.11 81.5) (xy 98.74 81.14) (xy 98.64 81.14)
 			)
 		)
