File: ControllerPCB/controller_pcb.kicad_pcb (KiCad board)
At the start: 2 copper layers, 67.1 x 59 mm, 11 parts, among them J1 USB3_A, U1 Pico, U3 AP63203WU

Commit message: half-done modifying controllerPCB
Parts:
- added H1: MountingHole, MountingHole:MountingHole_2.7mm, F.Cu at (64.1, 37.9)
- added H2: MountingHole, MountingHole:MountingHole_2.7mm, F.Cu at (64.1, 44.9)
- added H3: MountingHole, MountingHole:MountingHole_2.7mm, F.Cu at (64.1, 51.8)
- added H4: MountingHole, MountingHole:MountingHole_2.7mm, F.Cu at (64.1, 58.8)
- added PWR_SW1: SW_SPDT_BOX, switchbox_footprints:3_pin_header, F.Cu at (121.3, 92.2)
- U1: footprint MCU_RaspberryPi_and_Boards:RPi_Pico_SMD_TH -> Module:RaspberryPi_Pico_Common_THT
- U2: footprint Xbee:XBee -> switchbox_footprints:xbee
- moved U1 73.4 mm to (87.1, 66.8)
- moved J1 71.8 mm to (117.2, 69.0)
- moved C3 65.3 mm to (141.8, 128.4)
- moved C4 65.3 mm to (141.8, 131.7)
- moved L1 65.3 mm to (134.7, 130.6), turned to 0 degrees
- moved U3 51.8 mm to (141.5, 135.8)
- moved C2 48.9 mm to (146.6, 127.9), turned to 0 degrees
- moved R3 42.8 mm to (146.8, 133.2), turned to 0 degrees
- moved C1 42.2 mm to (150.9, 128.2)
- moved U2 42.2 mm to (146.8, 82.2)
- moved R_Buck_3 38.6 mm to (146.6, 130.5), turned to 0 degrees
Connections:
- C3 pad 1: Net-(U1-VSYS) -> Net-(PWR_SW1-B)
- C4 pad 1: Net-(U1-VSYS) -> Net-(PWR_SW1-B)
- L1 pad 2: Net-(U1-VSYS) -> Net-(PWR_SW1-C)
- U1 pad 39: Net-(U1-VSYS) -> Net-(PWR_SW1-B)
- U2 pad 1: Net-(U1-VSYS) -> Net-(PWR_SW1-B)
- U3 pad 1: Net-(U1-VSYS) -> Net-(PWR_SW1-C)
Routing:
- net Net-(U1-VSYS): track 64.9 -> 0.00 mm
- net Net-(U1-GPIO0): track 42.1 -> 0.00 mm
- net /DOUT: track 31.5 -> 0.00 mm
- net Net-(U3-SW): track 13.6 -> 0.00 mm
- net Net-(J1-VBUS): track 12.5 -> 0.00 mm
- net Net-(U3-EN): track 8.10 -> 0.00 mm
- net Net-(U3-BST): track 6.13 -> 0.00 mm
- removed copper zone on B.Cu, net GND
Other:
- board size 67.1 x 59 mm -> 81.3 x 82.1 mm
- board text removed: "GND"
