File: ControllerPCB/controller_pcb.kicad_pcb (KiCad board)
At the start: 2 copper layers, 81.3 x 82.1 mm, 16 parts, among them J1 USB3_A, U1 Pico, U3 AP63203WU

Commit message: series of changes
Parts:
- removed R3: 100k, Resistor_SMD:R_0805_2012Metric
- removed R_Buck_3: 100k, Resistor_SMD:R_0603_1608Metric
- removed U3: AP63203WU, Package_TO_SOT_SMD:TSOT-23-6
- added R3a1: 100k, Resistor_SMD:R_0805_2012Metric_Pad1.20x1.40mm_HandSolder, F.Cu at (109.3, 77.3)
- added R3b1: 100k, Resistor_SMD:R_0805_2012Metric_Pad1.20x1.40mm_HandSolder, F.Cu at (109.3, 72.9)
- added U2: AP63203WU, Package_TO_SOT_SMD:TSOT-23-6, F.Cu at (112.8, 75.3)
- C1: footprint Capacitor_SMD:C_0805_2012Metric -> switchbox_footprints:CAPC1005X70N
- C2: footprint Capacitor_SMD:C_0603_1608Metric -> switchbox_footprints:CAPC0603X33N
- C3, C4: footprint Capacitor_SMD:C_1206_3216Metric -> switchbox_footprints:CAPC3216X190N
- L1: footprint Inductor_SMD:L_6.3x6.3_H3 -> Inductor_SMD:L_0201_0603Metric_Pad0.64x0.40mm_HandSolder
- PWR_SW1: moved to B.Cu
- moved H1 82.7 mm to (130.6, 87.2)
- moved H4 79.6 mm to (124.3, 110.9)
- moved H2 69.1 mm to (119.2, 86.6)
- moved H3 69.1 mm to (119.2, 93.5)
- moved L1 62.6 mm to (112.9, 71.9), turned to 180 degrees
- moved C1 62.2 mm to (112.9, 78.9)
- moved C2 61.3 mm to (115.9, 74.9), turned to -90 degrees
- moved C3 60.9 mm to (117.4, 72.5), turned to 180 degrees
- moved C4 59.0 mm to (117.4, 78.0), turned to 180 degrees
- moved U2 27.5 mm to (124.0, 97.5)
- moved PWR_SW1 25.4 mm to (114.2, 67.9), turned to 180 degrees
- moved J1 16.5 mm to (132.0, 76.2), turned to 180 degrees
- moved U1 1.54 mm to (86.4, 65.4)
Connections:
- C1 pad 1: Net-(J1-VBUS) -> Sys_Vin
- C3 pad 1: Net-(PWR_SW1-B) -> 3.3VBuck
- C4 pad 1: Net-(PWR_SW1-B) -> 3.3VBuck
- L1 pad 2: Net-(PWR_SW1-C) -> 3.3VBuck
Routing:
- net 3.3VBuck: track 0.00 -> 8.32 mm
- net Net-(U2-SW): track 0.00 -> 6.41 mm
- net GND: track 0.00 -> 4.36 mm, vias 0 -> 4
- net Sys_Vin: track 0.00 -> 3.42 mm
- net Net-(U2-BST): track 0.00 -> 2.12 mm
- added copper zone on B.Cu, net GND
Other:
- board outline removed

Commit message: controller pcb
Parts:
- removed H1, H2, H3, H4: MountingHole, MountingHole:MountingHole_2.7mm
- removed R3a1, R3b1: 100k, Resistor_SMD:R_0805_2012Metric_Pad1.20x1.40mm_HandSolder
- removed the U2 at (112.8, 75.3)
- added D1: LED, switchbox_footprints:2_pin_header, F.Cu at (111.1, 87.0)
- added G***: LOGO, LOGO, F.Cu at (147.9, 110.6)
- added R1: 100, Capacitor_SMD:C_0603_1608Metric, F.Cu at (112.0, 80.3)
- added R3: 100k, Resistor_SMD:R_0805_2012Metric, F.Cu at (100.1, 91.5)
- added R_Buck_3: 100k, Resistor_SMD:R_0603_1608Metric, F.Cu at (97.0, 84.3)
- added U3: AP63203WU, Package_TO_SOT_SMD:TSOT-23-6, F.Cu at (93.2, 84.2)
- C1: footprint switchbox_footprints:CAPC1005X70N -> Capacitor_SMD:C_1206_3216Metric_Pad1.33x1.80mm_HandSolder
- C2: footprint switchbox_footprints:CAPC0603X33N -> Capacitor_SMD:C_0603_1608Metric_Pad1.08x0.95mm_HandSolder
- C3, C4: footprint switchbox_footprints:CAPC3216X190N -> Capacitor_SMD:C_0603_1608Metric_Pad1.08x0.95mm_HandSolder
- L1: footprint Inductor_SMD:L_0201_0603Metric_Pad0.64x0.40mm_HandSolder -> Inductor_SMD:L_6.3x6.3_H3
- PWR_SW1: moved to F.Cu
- moved U1 49.2 mm to (93.6, 114.1), turned to 90 degrees
- moved J1 28.6 mm to (103.9, 71.0), turned to -90 degrees
- moved C3 26.6 mm to (97.0, 89.5), turned to 90 degrees
- moved C4 25.2 mm to (95.0, 89.5), turned to 90 degrees
- moved C1 23.7 mm to (92.0, 90.0), turned to -90 degrees
- moved C2 20.4 mm to (104.1, 91.5), turned to 0 degrees
- moved U2 19.6 mm to (133.6, 80.4), turned to -90 degrees
- moved L1 17.9 mm to (102.2, 86.2)
- moved PWR_SW1 6.22 mm to (111.2, 73.3), turned to 90 degrees
Connections:
- C1 pad 1: Sys_Vin -> Net-(J1-VBUS)
- C3 pad 1: 3.3VBuck -> Net-(PWR_SW1-B)
- C4 pad 1: 3.3VBuck -> Net-(PWR_SW1-B)
- L1 pad 2: 3.3VBuck -> Net-(PWR_SW1-C)
Routing:
- net Net-(PWR_SW1-B): track 0.00 -> 73.3 mm
- net Net-(U1-GPIO0): track 0.00 -> 64.7 mm
- net /DOUT: track 0.00 -> 62.3 mm
- net Net-(J1-VBUS): track 0.00 -> 32.1 mm, vias 0 -> 2
- net Net-(PWR_SW1-C): track 0.00 -> 22.4 mm
- net Net-(U3-SW): track 6.41 -> 26.2 mm, vias 0 -> 2
- net Net-(U3-EN): track 0.00 -> 14.2 mm, vias 0 -> 2
- net Net-(U3-BST): track 2.12 -> 16.1 mm, vias 0 -> 2
- net 3.3VBuck: track 8.32 -> 0.00 mm
- net Net-(D1-A): track 0.00 -> 8.05 mm
- net Sys_Vin: track 3.42 -> 0.00 mm
- net GND: track 4.36 -> 6.98 mm, vias 4 -> 5
Other:
- board outline added: 62.8 x 51.2 mm
- board text added: "Controller PCB SP26 Ludvig Fellstrom Linnea Furlan"
- board text added: "Pico W"

Commit message: jlc files
Parts:
- added H1: MountingHole, MountingHole:MountingHole_3.2mm_M3, F.Cu at (120.0, 75.0)
- added H2: MountingHole, MountingHole:MountingHole_3.2mm_M3, F.Cu at (148.0, 113.0)
- moved G*** 3.65 mm to (147.9, 107.0)
Routing:
- added copper zone on F.Cu, net (none)
Changed lines of the file:
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@@
 		(sheetname "/")
 		(sheetfile "controller_pcb.kicad_sch")
-		(attr smd)
+		(attr smd exclude_from_pos_files exclude_from_bom)
 		(fp_line
 			(start 5.15 -3.275)
@@
 		(sheetname "/")
 		(sheetfile "controller_pcb.kicad_sch")
-		(attr smd)
+		(attr smd exclude_from_pos_files exclude_from_bom)
 		(fp_line
 			(start -13 19)
@@
 		)
 	)
+	(footprint "MountingHole:MountingHole_3.2mm_M3"
+		(layer "F.Cu")
+		(at 120 75)
+		(descr "Mounting Hole 3.2mm, M3, no annular, generated by kicad-footprint-generator mountinghole.py")
+		(tags "mountinghole M3")
+		(property "Reference" "H1"
+			(at 0 -4.15 0)
+			(layer "F.SilkS")
+			(hide yes)
+			(effects
+				(font
+					(size 1 1)
+					(thickness 0.15)
+				)
+			)
+		)
+		(property "Value" "MountingHole"
+			(at 0 4.15 0)
+			(layer "F.Fab")
+			(hide yes)
+			(effects
+				(font
+					(size 1 1)
+					(thickness 0.15)
+				)
+			)
+		)
+		(property "Datasheet" "~"
+			(at 0 0 0)
+			(layer "F.Fab")
+			(hide yes)
+			(effects
+				(font
+					(size 1.27 1.27)
+					(thickness 0.15)
+				)
+			)
+		)
+		(property "Description" "Mounting Hole without connection"
+			(at 0 0 0)
+			(layer "F.Fab")
+			(hide yes)
+			(effects
+				(font
+					(size 1.27 1.27)
+					(thickness 0.15)
+				)
+			)
+		)
+		(property ki_fp_filters "MountingHole*")
+		(sheetname "/")
+		(sheetfile "controller_pcb.kicad_sch")
+		(attr exclude_from_pos_files exclude_from_bom)
+		(fp_circle
+			(center 0 0)
+			(end 3.2 0)
+			(stroke
+				(width 0.15)
+				(type solid)
+			)
+			(fill no)
+			(layer "Cmts.User")
+		)
+		(fp_circle
+			(center 0 0)
+			(end 3.45 0)
+			(stroke
+				(width 0.05)
+				(type solid)
+			)
+			(fill no)
+			(layer "F.CrtYd")
+		)
+		(fp_text user "${REFERENCE}"
+			(at 0 0 0)
+			(layer "F.Fab")
+			(effects
+				(font
+					(size 1 1)
+					(thickness 0.15)
+				)
+			)
+		)
+		(pad "" np_thru_hole circle
+			(at 0 0)
+			(size 3.2 3.2)
+			(drill 3.2)
+			(layers "*.Cu" "*.Mask")
+		)
+		(embedded_fonts no)
+	)
 	(footprint "Capacitor_SMD:C_1206_3216Metric_Pad1.33x1.80mm_HandSolder"
 		(layer "F.Cu")
@@
 		(sheetname "/")
 		(sheetfile "controller_pcb.kicad_sch")
-		(attr through_hole)
+		(attr through_hole exclude_from_pos_files exclude_from_bom)
 		(fp_line
 			(start 13 -2.78)
@@
 		(sheetname "/")
 		(sheetfile "controller_pcb.kicad_sch")
-		(attr smd)
+		(attr smd exclude_from_pos_files exclude_from_bom)
 		(fp_line
 			(start 4.15 -3.25)
@@
 	(footprint "LOGO"
 		(layer "F.Cu")
-		(at 147.903049 110.648614 90)
+		(at 147.903049 107 90)
 		(property "Reference" "G***"
 			(at 0 0 90)
@@
 		(sheetname "/")
 		(sheetfile "controller_pcb.kicad_sch")
-		(attr through_hole)
+		(attr through_hole exclude_from_pos_files exclude_from_bom)
 		(fp_line
 			(start -3.51 6.65)
@@
 		)
 	)
+	(footprint "MountingHole:MountingHole_3.2mm_M3"
+		(layer "F.Cu")
+		(at 148 113)
+		(descr "Mounting Hole 3.2mm, M3, no annular, generated by kicad-footprint-generator mountinghole.py")
+		(tags "mountinghole M3")
+		(property "Reference" "H2"
+			(at 0 -4.15 0)
+			(layer "F.SilkS")
+			(hide yes)
+			(effects
+				(font
+					(size 1 1)
+					(thickness 0.15)
+				)
+			)
+		)
+		(property "Value" "MountingHole"
+			(at 0 4.15 0)
+			(layer "F.Fab")
+			(hide yes)
+			(effects
+				(font
+					(size 1 1)
+					(thickness 0.15)
+				)
+			)
+		)
+		(property "Datasheet" "~"
+			(at 0 0 0)
+			(layer "F.Fab")
+			(hide yes)
+			(effects
+				(font
+					(size 1.27 1.27)
+					(thickness 0.15)
+				)
+			)
+		)
+		(property "Description" "Mounting Hole without connection"
+			(at 0 0 0)
+			(layer "F.Fab")
+			(hide yes)
+			(effects
+				(font
+					(size 1.27 1.27)
+					(thickness 0.15)
+				)
+			)
+		)
+		(property ki_fp_filters "MountingHole*")
+		(sheetname "/")
+		(sheetfile "controller_pcb.kicad_sch")
+		(attr exclude_from_pos_files exclude_from_bom)
+		(fp_circle
+			(center 0 0)
+			(end 3.2 0)
+			(stroke
+				(width 0.15)
+				(type solid)
+			)
+			(fill no)
+			(layer "Cmts.User")
+		)
+		(fp_circle
+			(center 0 0)
+			(end 3.45 0)
+			(stroke
+				(width 0.05)
+				(type solid)
+			)
+			(fill no)
+			(layer "F.CrtYd")
+		)
+		(fp_text user "${REFERENCE}"
+			(at 0 0 0)
+			(layer "F.Fab")
+			(effects
+				(font
+					(size 1 1)
+					(thickness 0.15)
+				)
+			)
+		)
+		(pad "" np_thru_hole circle
+			(at 0 0)
+			(size 3.2 3.2)
+			(drill 3.2)
+			(layers "*.Cu" "*.Mask")
+		)
+		(embedded_fonts no)
+	)
 	(footprint "Capacitor_SMD:C_0603_1608Metric_Pad1.08x0.95mm_HandSolder"
 		(layer "F.Cu")
@@
 	)
 	(gr_text "Controller PCB\nSP26\nLudvig Fellstrom\nLinnea Furlan"
-		(at 150.625 107.5 90)
+		(at 150.625 104.5 90)
 		(layer "F.SilkS")
 		(effects
@@
 	)
 	(zone
+		(net 0)
+		(net_name "")
+		(layer "F.Cu")
+		(hatch edge 0.5)
+		(priority 1)
+		(connect_pads
+			(clearance 0.5)
+		)
+		(min_thickness 0.25)
+		(filled_areas_thickness no)
+		(fill yes
+			(thermal_gap 0.5)
+			(thermal_bridge_width 0.5)
+			(island_removal_mode 1)
+			(island_area_min 10)
+		)
+		(polygon
+			(pts
+				(xy 89.5 66) (xy 152.5 66) (xy 152.5 117.5) (xy 90 117.5)
+			)
+		)
+	)
+	(zone
