File: ControllerPCB/controller_pcb.kicad_sch (KiCad schematic)
At the start: 2 parts, among them U1 Pico

Commit message: Idk what happened last time
Parts:
- added C1: 10µF, Capacitor_SMD:C_0805_2012Metric, symbol Device:C
- added C2: 0.1µF, Capacitor_SMD:C_0603_1608Metric, symbol Device:C
- added C3, C4: 22µF, Capacitor_SMD:C_1206_3216Metric, symbol Device:C
- added J1: USB3_A, Connector_USB:USB3_A_Molex_48393-001, symbol Connector:USB3_A
- added L1: 4.7µH, Inductor_SMD:L_6.3x6.3_H3, symbol Device:L
- added R3: 100k, Resistor_SMD:R_0805_2012Metric, symbol Device:R
- added R_Buck_3: 100k, Resistor_SMD:R_0603_1608Metric, symbol Device:R
- added U3: AP63203WU, Package_TO_SOT_SMD:TSOT-23-6, symbol Regulator_Switching:AP63203WU
- U1: footprint RPi_Pico:RPi_Pico_SMD_TH -> MCU_RaspberryPi_and_Boards:RPi_Pico_SMD_TH
- U2: footprint (none) -> Xbee:XBee
Connections:
- net GND: now also U1.13 (GND), U1.18 (GND), U1.23 (GND), U1.28 (GND), U1.3 (GND), U1.38 (GND), U1.42 (GND), U1.8 (GND), C1.2, C3.2, C4.2, J1.10 (SHIELD), J1.4 (GND), J1.7 (DRAIN), R_Buck_3.2, U3.4 (GND)
- net at U1.39 (VSYS): now also U2.1 (VCC), C3.1, C4.1, L1.2, U3.1 (FB)
- new net: C1.1, J1.1 (VBUS), R3.2, U3.3 (IN)
- new net: C2.2, L1.1, U3.5 (SW)
- new net: R3.1, R_Buck_3.1, U3.2 (EN)
- new net: C2.1, U3.6 (BST)
- no-connect marks 0 -> 54

Commit message: half-done modifying controllerPCB
Parts:
- added H1, H2, H3, H4: MountingHole, MountingHole:MountingHole_2.7mm, symbol Mechanical:MountingHole
- added PWR_SW1: SW_SPDT_BOX, switchbox_footprints:3_pin_header, symbol Switch:SW_Push_SPDT
- U1: footprint MCU_RaspberryPi_and_Boards:RPi_Pico_SMD_TH -> Module:RaspberryPi_Pico_Common_THT
- U2: footprint Xbee:XBee -> switchbox_footprints:xbee
Connections:
- net GND: now also PWR_SW1.1 (A)
- net at C3.1, C4.1, U1.39 (VSYS)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: now also PWR_SW1.2 (B); no longer L1.2, U3.1 (FB)
- new net: L1.2, PWR_SW1.3 (C), U3.1 (FB)
Other:
- moved on the sheet: C1, C2, C3, C4, J1, L1, R3, R_Buck_3, U1, U2, U3
